Commit message: First try of building grasp env for training

File: source/gen3/gen3_2f85/gen3_2f85_fixed.urdf (robot description, URDF)
Before this commit: robot gen3_, 31 links, 30 joints
Joints:
- joint gen3_robotiq_85_left_finger_tip_joint: limit (none) -> lower=-0.8 upper=0.0 effort=50 velocity=0.5; type continuous -> revolute
- joint gen3_robotiq_85_left_inner_knuckle_joint: limit (none) -> lower=0.0 upper=0.8 effort=50 velocity=0.5; type continuous -> revolute
- joint gen3_robotiq_85_right_finger_tip_joint: limit (none) -> lower=0.0 upper=0.8 effort=50 velocity=0.5; type continuous -> revolute
- joint gen3_robotiq_85_right_inner_knuckle_joint: limit (none) -> lower=-0.8 upper=0.0 effort=50 velocity=0.5; type continuous -> revolute
